File: layer1/layer1v2.sch (EAGLE design)
At the start: 7 parts, among them U1 microSD, U2 DS3234

Commit message: I don't know why eagles file thing hates me, but here we are
Parts:
- added C2, C3: 0.1uF, SparkFun:CAP0402-CAP
- added C4: 4.7uF, SparkFun:CAP0402-CAP
- added J3: (no value), SparkFun-Connectors:M02LOCK
- added R2, R3, R4: 10k, SparkFun:RESISTOR0402-RES
- added U3: MMA8452Q, SparkFun:MMA8452Q
Connections:
- new net BYP: C3.1, U3.BYP
- new net SA0: R4.1, U3.SA0
- new net SCL: J3.2, R2.1, U3.SCL
- new net SDA: J3.1, R3.1, U3.SDA
- net GND: now also C2.2, C3.2, C4.2, U3.GND@0, U3.GND@1, U3.GND@2
- net VCC: now also C2.1, C4.1, R2.2, R3.2, R4.2, U3.VDD, U3.VDDIO
Other:
- note added: "Jumper open by default, so SA0 = 0"
Changed lines of the file:
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@@
 <part name="J1" library="SparkFun-Connectors" deviceset="M12" device="PTH"/>
 <part name="J2" library="SparkFun-Connectors" deviceset="M12" device="PTH"/>
+<part name="U3" library="SparkFun" deviceset="MMA8452Q" device=""/>
+<part name="C2" library="SparkFun" deviceset="CAP" device="0402-CAP" value="0.1uF"/>
+<part name="C3" library="SparkFun" deviceset="CAP" device="0402-CAP" value="0.1uF"/>
+<part name="C4" library="SparkFun" deviceset="CAP" device="0402-CAP" value="4.7uF"/>
+<part name="R2" library="SparkFun" deviceset="RESISTOR" device="0402-RES" value="10k"/>
+<part name="R3" library="SparkFun" deviceset="RESISTOR" device="0402-RES" value="10k"/>
+<part name="GND3" library="SparkFun" deviceset="GND" device=""/>
+<part name="R4" library="SparkFun" deviceset="RESISTOR" device="0402-RES" value="10k"/>
+<part name="J3" library="SparkFun-Connectors" deviceset="M02" device="LOCK"/>
 </parts>
 <sheets>
@@
 <text x="139.954" y="145.288" size="1.778" layer="97" rot="R180">Connection to 3.7V System</text>
 <text x="109.22" y="101.6" size="1.778" layer="97" rot="R90">Lipo Battery</text>
+<text x="193.04" y="27.94" size="1.778" layer="97">Jumper open by default, so SA0 = 0</text>
 </plain>
 <instances>
@@
 <instance part="J1" gate="G$1" x="50.8" y="33.02"/>
 <instance part="J2" gate="G$1" x="99.06" y="30.48" rot="R180"/>
+<instance part="U3" gate="G$1" x="147.32" y="43.18"/>
+<instance part="C2" gate="G$1" x="106.68" y="38.1"/>
+<instance part="C3" gate="G$1" x="127" y="38.1"/>
+<instance part="C4" gate="G$1" x="116.84" y="38.1"/>
+<instance part="R2" gate="G$1" x="165.1" y="58.42" rot="R90"/>
+<instance part="R3" gate="G$1" x="172.72" y="58.42" rot="R90"/>
+<instance part="GND3" gate="1" x="134.62" y="25.4"/>
+<instance part="R4" gate="G$1" x="187.96" y="43.18" rot="R90"/>
+<instance part="J3" gate="G$1" x="73.66" y="53.34"/>
 </instances>
 <busses>
@@
 <label x="81.28" y="38.1" size="1.778" layer="95"/>
 <pinref part="J2" gate="G$1" pin="4"/>
+</segment>
+<segment>
+<wire x1="165.1" y1="66.04" x2="165.1" y2="63.5" width="0.1524" layer="91"/>
+<pinref part="R2" gate="G$1" pin="2"/>
+<label x="165.1" y="66.04" size="1.778" layer="95" rot="R270"/>
+</segment>
+<segment>
+<wire x1="172.72" y1="66.04" x2="172.72" y2="63.5" width="0.1524" layer="91"/>
+<pinref part="R3" gate="G$1" pin="2"/>
+<label x="172.72" y="66.04" size="1.778" layer="95" rot="R270"/>
+</segment>
+<segment>
+<wire x1="137.16" y1="50.8" x2="134.62" y2="50.8" width="0.1524" layer="91"/>
+<wire x1="137.16" y1="48.26" x2="134.62" y2="48.26" width="0.1524" layer="91"/>
+<wire x1="134.62" y1="48.26" x2="134.62" y2="50.8" width="0.1524" layer="91"/>
+<wire x1="116.84" y1="43.18" x2="116.84" y2="48.26" width="0.1524" layer="91"/>
+<wire x1="116.84" y1="48.26" x2="134.62" y2="48.26" width="0.1524" layer="91"/>
+<wire x1="106.68" y1="43.18" x2="106.68" y2="48.26" width="0.1524" layer="91"/>
+<wire x1="106.68" y1="48.26" x2="116.84" y2="48.26" width="0.1524" layer="91"/>
+<junction x="134.62" y="48.26"/>
+<junction x="116.84" y="48.26"/>
+<pinref part="U3" gate="G$1" pin="VDD"/>
+<pinref part="U3" gate="G$1" pin="VDDIO"/>
+<pinref part="C4" gate="G$1" pin="1"/>
+<pinref part="C2" gate="G$1" pin="1"/>
+<wire x1="134.62" y1="50.8" x2="134.62" y2="58.42" width="0.1524" layer="91"/>
+<junction x="134.62" y="50.8"/>
+<label x="134.62" y="58.42" size="1.778" layer="95" rot="R270"/>
+</segment>
+<segment>
+<wire x1="187.96" y1="50.8" x2="187.96" y2="48.26" width="0.1524" layer="91"/>
+<pinref part="R4" gate="G$1" pin="2"/>
+<label x="187.96" y="50.8" size="1.778" layer="95" rot="R270"/>
 </segment>
 </net>
@@
 <pinref part="J2" gate="G$1" pin="2"/>
 </segment>
+<segment>
+<wire x1="137.16" y1="35.56" x2="134.62" y2="35.56" width="0.1524" layer="91"/>
+<wire x1="134.62" y1="35.56" x2="134.62" y2="33.02" width="0.1524" layer="91"/>
+<wire x1="134.62" y1="33.02" x2="134.62" y2="27.94" width="0.1524" layer="91"/>
+<wire x1="137.16" y1="38.1" x2="134.62" y2="38.1" width="0.1524" layer="91"/>
+<wire x1="134.62" y1="38.1" x2="134.62" y2="35.56" width="0.1524" layer="91"/>
+<wire x1="137.16" y1="40.64" x2="134.62" y2="40.64" width="0.1524" layer="91"/>
+<wire x1="134.62" y1="40.64" x2="134.62" y2="38.1" width="0.1524" layer="91"/>
+<wire x1="106.68" y1="35.56" x2="106.68" y2="33.02" width="0.1524" layer="91"/>
+<wire x1="106.68" y1="33.02" x2="116.84" y2="33.02" width="0.1524" layer="91"/>
+<wire x1="116.84" y1="35.56" x2="116.84" y2="33.02" width="0.1524" layer="91"/>
+<wire x1="116.84" y1="33.02" x2="127" y2="33.02" width="0.1524" layer="91"/>
+<wire x1="127" y1="33.02" x2="134.62" y2="33.02" width="0.1524" layer="91"/>
+<wire x1="127" y1="35.56" x2="127" y2="33.02" width="0.1524" layer="91"/>
+<junction x="134.62" y="35.56"/>
+<junction x="134.62" y="38.1"/>
+<junction x="116.84" y="33.02"/>
+<junction x="134.62" y="33.02"/>
+<junction x="127" y="33.02"/>
+<pinref part="U3" gate="G$1" pin="GND@0"/>
+<pinref part="GND3" gate="1" pin="GND"/>
+<pinref part="U3" gate="G$1" pin="GND@1"/>
+<pinref part="U3" gate="G$1" pin="GND@2"/>
+<pinref part="C2" gate="G$1" pin="2"/>
+<pinref part="C4" gate="G$1" pin="2"/>
+<pinref part="C3" gate="G$1" pin="2"/>
+</segment>
 </net>
 <net name="MISO" class="0">
@@
 </segment>
 </net>
+<net name="BYP" class="0">
+<segment>
+<wire x1="137.16" y1="45.72" x2="127" y2="45.72" width="0.1524" layer="91"/>
+<wire x1="127" y1="45.72" x2="127" y2="43.18" width="0.1524" layer="91"/>
+<pinref part="U3" gate="G$1" pin="BYP"/>
+<pinref part="C3" gate="G$1" pin="1"/>
+</segment>
+</net>
+<net name="SCL" class="0">
+<segment>
+<wire x1="160.02" y1="50.8" x2="165.1" y2="50.8" width="0.1524" layer="91"/>
+<wire x1="165.1" y1="50.8" x2="165.1" y2="53.34" width="0.1524" layer="91"/>
+<wire x1="165.1" y1="50.8" x2="180.34" y2="50.8" width="0.1524" layer="91"/>
+<junction x="165.1" y="50.8"/>
+<label x="175.26" y="50.8" size="1.778" layer="95"/>
+<pinref part="U3" gate="G$1" pin="SCL"/>
+<pinref part="R2" gate="G$1" pin="1"/>
+</segment>
+<segment>
+<pinref part="J3" gate="G$1" pin="2"/>
+<wire x1="81.28" y1="55.88" x2="86.36" y2="55.88" width="0.1524" layer="91"/>
+<label x="81.28" y="55.88" size="1.778" layer="95"/>
+</segment>
+</net>
+<net name="SDA" class="0">
+<segment>
+<wire x1="160.02" y1="48.26" x2="172.72" y2="48.26" width="0.1524" layer="91"/>
+<wire x1="172.72" y1="48.26" x2="172.72" y2="53.34" width="0.1524" layer="91"/>
+<wire x1="172.72" y1="48.26" x2="180.34" y2="48.26" width="0.1524" layer="91"/>
+<junction x="172.72" y="48.26"/>
+<label x="175.26" y="48.26" size="1.778" layer="95"/>
+<pinref part="U3" gate="G$1" pin="SDA"/>
+<pinref part="R3" gate="G$1" pin="1"/>
+</segment>
+<segment>
+<pinref part="J3" gate="G$1" pin="1"/>
+<wire x1="81.28" y1="53.34" x2="86.36" y2="53.34" width="0.1524" layer="91"/>
+<label x="81.28" y="53.34" size="1.778" layer="95"/>
+</segment>
+</net>
+<net name="SA0" class="0">
+<segment>
+<wire x1="160.02" y1="35.56" x2="187.96" y2="35.56" width="0.1524" layer="91"/>
+<wire x1="187.96" y1="35.56" x2="187.96" y2="38.1" width="0.1524" layer="91"/>
+<label x="162.56" y="35.56" size="1.778" layer="95"/>
+<pinref part="U3" gate="G$1" pin="SA0"/>
+<pinref part="R4" gate="G$1" pin="1"/>
+</segment>
+</net>
