File: layer1/layer1v2.brd (EAGLE design)
At the start: 17.8 x 48.3 mm, 7 parts, among them U1 microSD, U2 DS3234

Commit message: I don't know why eagles file thing hates me, but here we are
Parts:
- added C2, C3: 0.1uF, SparkFun:0402-CAP
- added C4: 4.7uF, SparkFun:0402-CAP
- added J3: (no value), SparkFun-Connectors:1X02_LOCK
- added R2, R3, R4: 10k, SparkFun:0402-RES
- added U3: MMA8452Q, SparkFun:QFN-16_0.5MM
- moved U2 15.2 mm to (8.89, 7.62)
Connections:
- new net BYP: C3.1, U3.2
- new net SA0: R4.1, U3.7
- new net SCL: J3.2, R2.1, U3.4
- new net SDA: J3.1, R3.1, U3.6
- net GND: now also C2.2, C3.2, C4.2, U3.10, U3.12, U3.5
- net VCC: now also C2.1, C4.1, R2.2, R3.2, R4.2, U3.1, U3.14
Changed lines of the file:
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@@
 <element name="R1" library="SparkFun" package="0402-RES" value="10k" x="3.81" y="15.24" rot="R90"/>
 <element name="U1" library="SparkFun" package="MICRO-SD-SOCKET-PP" value="microSD" x="15.24" y="30.48"/>
-<element name="U2" library="SparkFun" package="DS3234" value="DS3234" x="8.89" y="22.86" rot="R270"/>
+<element name="U2" library="SparkFun" package="DS3234" value="DS3234" x="8.89" y="7.62" rot="R270"/>
 <element name="J1" library="SparkFun-Connectors" package="1X12" value="" x="1.27" y="1.27" rot="R90"/>
 <element name="J2" library="SparkFun-Connectors" package="1X12" value="" x="16.51" y="29.21" rot="R270"/>
+<element name="U3" library="SparkFun" package="QFN-16_0.5MM" value="MMA8452Q" x="0" y="-3.81"/>
+<element name="C2" library="SparkFun" package="0402-CAP" value="0.1uF" x="0" y="-8.89"/>
+<element name="C3" library="SparkFun" package="0402-CAP" value="0.1uF" x="3.81" y="-8.89"/>
+<element name="C4" library="SparkFun" package="0402-CAP" value="4.7uF" x="0" y="-12.7"/>
+<element name="R2" library="SparkFun" package="0402-RES" value="10k" x="3.81" y="-12.7"/>
+<element name="R3" library="SparkFun" package="0402-RES" value="10k" x="0" y="-16.51"/>
+<element name="R4" library="SparkFun" package="0402-RES" value="10k" x="3.81" y="-16.51"/>
+<element name="J3" library="SparkFun-Connectors" package="1X02_LOCK" value="" x="0" y="-22.86"/>
 </elements>
 <signals>
@@
 <contactref element="U1" pad="4"/>
 <contactref element="J2" pad="4"/>
-<wire x1="4.205" y1="24.765" x2="9.6" y2="41.38" width="0" layer="19" extent="1-1"/>
-<wire x1="3.81" y1="14.59" x2="4.205" y2="24.765" width="0" layer="19" extent="1-1"/>
+<contactref element="R2" pad="2"/>
+<contactref element="R3" pad="2"/>
+<contactref element="U3" pad="14"/>
+<contactref element="U3" pad="1"/>
+<contactref element="C4" pad="1"/>
+<contactref element="C2" pad="1"/>
+<contactref element="R4" pad="2"/>
+<wire x1="4.205" y1="9.525" x2="9.6" y2="41.38" width="0" layer="19" extent="1-1"/>
+<wire x1="3.81" y1="14.59" x2="4.205" y2="9.525" width="0" layer="19" extent="1-1"/>
 <wire x1="13.97" y1="14.59" x2="3.81" y2="14.59" width="0" layer="19" extent="1-1"/>
 <wire x1="16.51" y1="21.59" x2="13.97" y2="14.59" width="0" layer="19" extent="1-1"/>
+<wire x1="0.5" y1="-2.535" x2="3.81" y2="14.59" width="0" layer="19" extent="1-1"/>
+<wire x1="-1.275" y1="-2.81" x2="0.5" y2="-2.535" width="0" layer="19" extent="1-1"/>
+<wire x1="-0.65" y1="-8.89" x2="-1.275" y2="-2.81" width="0" layer="19" extent="1-1"/>
+<wire x1="-0.65" y1="-12.7" x2="-0.65" y2="-8.89" width="0" layer="19" extent="1-1"/>
+<wire x1="0.65" y1="-16.51" x2="-0.65" y2="-12.7" width="0" layer="19" extent="1-1"/>
+<wire x1="4.46" y1="-16.51" x2="0.65" y2="-16.51" width="0" layer="19" extent="1-1"/>
+<wire x1="4.46" y1="-12.7" x2="4.46" y2="-16.51" width="0" layer="19" extent="1-1"/>
 </signal>
 <signal name="GND">
@@
 <contactref element="J1" pad="9"/>
 <contactref element="J2" pad="2"/>
+<contactref element="U3" pad="5"/>
+<contactref element="U3" pad="10"/>
+<contactref element="U3" pad="12"/>
+<contactref element="C2" pad="2"/>
+<contactref element="C4" pad="2"/>
+<contactref element="C3" pad="2"/>
 <wire x1="11.8" y1="41.38" x2="14.79" y2="44.03" width="0" layer="19" extent="1-1"/>
+<wire x1="11.43" y1="39.37" x2="11.8" y2="41.38" width="0" layer="19" extent="1-16"/>
 <wire x1="1.64" y1="45.03" x2="11.8" y2="41.38" width="0" layer="19" extent="1-1"/>
-<wire x1="16.51" y1="26.67" x2="11.8" y2="41.38" width="0" layer="19" extent="1-1"/>
-<wire x1="13.575" y1="22.225" x2="16.51" y2="26.67" width="0" layer="19" extent="1-1"/>
-<wire x1="13.575" y1="20.955" x2="13.575" y2="22.225" width="0" layer="19" extent="1-1"/>
-<wire x1="13.575" y1="19.685" x2="13.575" y2="20.955" width="0" layer="19" extent="1-1"/>
-<wire x1="13.575" y1="18.415" x2="13.575" y2="19.685" width="0" layer="19" extent="1-1"/>
-<wire x1="13.575" y1="17.145" x2="13.575" y2="18.415" width="0" layer="19" extent="1-1"/>
-<wire x1="13.97" y1="15.89" x2="13.575" y2="17.145" width="0" layer="19" extent="1-1"/>
-<wire x1="11.43" y1="39.37" x2="13.575" y2="22.225" width="0" layer="19" extent="1-16"/>
-<wire x1="4.205" y1="20.955" x2="11.43" y2="39.37" width="0" layer="19" extent="1-16"/>
-<wire x1="4.205" y1="19.685" x2="4.205" y2="20.955" width="0" layer="19" extent="1-1"/>
-<wire x1="4.205" y1="18.415" x2="4.205" y2="19.685" width="0" layer="19" extent="1-1"/>
-<wire x1="4.205" y1="17.145" x2="4.205" y2="18.415" width="0" layer="19" extent="1-1"/>
-<wire x1="1.27" y1="21.59" x2="4.205" y2="20.955" width="0" layer="19" extent="1-1"/>
-<wire x1="4.205" y1="27.305" x2="4.205" y2="20.955" width="0" layer="19" extent="1-1"/>
+<wire x1="16.51" y1="26.67" x2="11.43" y2="39.37" width="0" layer="19" extent="16-16"/>
+<wire x1="13.575" y1="6.985" x2="16.51" y2="26.67" width="0" layer="19" extent="1-1"/>
+<wire x1="13.575" y1="5.715" x2="13.575" y2="6.985" width="0" layer="19" extent="1-1"/>
+<wire x1="13.575" y1="4.445" x2="13.575" y2="5.715" width="0" layer="19" extent="1-1"/>
+<wire x1="13.575" y1="3.175" x2="13.575" y2="4.445" width="0" layer="19" extent="1-1"/>
+<wire x1="13.575" y1="1.905" x2="13.575" y2="3.175" width="0" layer="19" extent="1-1"/>
+<wire x1="13.97" y1="15.89" x2="13.575" y2="1.905" width="0" layer="19" extent="1-1"/>
+<wire x1="4.205" y1="5.715" x2="13.575" y2="5.715" width="0" layer="19" extent="1-1"/>
+<wire x1="4.205" y1="4.445" x2="4.205" y2="5.715" width="0" layer="19" extent="1-1"/>
+<wire x1="4.205" y1="3.175" x2="4.205" y2="4.445" width="0" layer="19" extent="1-1"/>
+<wire x1="4.205" y1="1.905" x2="4.205" y2="3.175" width="0" layer="19" extent="1-1"/>
+<wire x1="1.27" y1="21.59" x2="4.205" y2="5.715" width="0" layer="19" extent="1-1"/>
+<wire x1="4.205" y1="12.065" x2="4.205" y2="5.715" width="0" layer="19" extent="1-1"/>
+<wire x1="1.275" y1="-3.31" x2="4.205" y2="1.905" width="0" layer="19" extent="1-1"/>
+<wire x1="1.275" y1="-4.31" x2="1.275" y2="-3.31" width="0" layer="19" extent="1-1"/>
+<wire x1="-1.275" y1="-4.81" x2="1.275" y2="-4.31" width="0" layer="19" extent="1-1"/>
+<wire x1="0.65" y1="-8.89" x2="-1.275" y2="-4.81" width="0" layer="19" extent="1-1"/>
+<wire x1="0.65" y1="-12.7" x2="0.65" y2="-8.89" width="0" layer="19" extent="1-1"/>
+<wire x1="4.46" y1="-8.89" x2="0.65" y2="-8.89" width="0" layer="19" extent="1-1"/>
 </signal>
 <signal name="MISO">
@@
 <contactref element="J2" pad="10"/>
 <wire x1="12.9" y1="41.18" x2="16.51" y2="6.35" width="0" layer="19" extent="1-1"/>
-<wire x1="13.575" y1="27.305" x2="12.9" y2="41.18" width="0" layer="19" extent="1-1"/>
+<wire x1="13.575" y1="12.065" x2="12.9" y2="41.18" width="0" layer="19" extent="1-1"/>
 </signal>
 <signal name="MOSI">
@@
 <contactref element="J2" pad="11"/>
 <wire x1="8.5" y1="41.18" x2="16.51" y2="3.81" width="0" layer="19" extent="1-1"/>
-<wire x1="13.575" y1="24.765" x2="8.5" y2="41.18" width="0" layer="19" extent="1-1"/>
+<wire x1="13.575" y1="9.525" x2="8.5" y2="41.18" width="0" layer="19" extent="1-1"/>
 </signal>
 <signal name="INT/SQW">
@@
 <contactref element="U2" pad="5"/>
 <contactref element="J1" pad="8"/>
-<wire x1="4.205" y1="23.495" x2="3.81" y2="15.89" width="0" layer="19" extent="1-1"/>
-<wire x1="1.27" y1="19.05" x2="4.205" y2="23.495" width="0" layer="19" extent="1-1"/>
+<wire x1="4.205" y1="8.255" x2="3.81" y2="15.89" width="0" layer="19" extent="1-1"/>
+<wire x1="1.27" y1="19.05" x2="4.205" y2="8.255" width="0" layer="19" extent="1-1"/>
 </signal>
 <signal name="VBATT">
 <contactref element="U2" pad="16"/>
 <contactref element="BAT1" pad="PWR@1"/>
-<wire x1="11.43" y1="31.496" x2="13.575" y2="23.495" width="0" layer="19" extent="1-1"/>
+<wire x1="11.43" y1="31.496" x2="13.575" y2="8.255" width="0" layer="19" extent="1-1"/>
 </signal>
 <signal name="SD_CS">
@@
 <contactref element="J2" pad="9"/>
 <wire x1="10.7" y1="41.18" x2="16.51" y2="8.89" width="0" layer="19" extent="1-1"/>
-<wire x1="13.575" y1="26.035" x2="10.7" y2="41.18" width="0" layer="19" extent="1-1"/>
-<wire x1="13.575" y1="28.575" x2="13.575" y2="26.035" width="0" layer="19" extent="1-1"/>
+<wire x1="13.575" y1="10.795" x2="10.7" y2="41.18" width="0" layer="19" extent="1-1"/>
+<wire x1="13.575" y1="13.335" x2="13.575" y2="10.795" width="0" layer="19" extent="1-1"/>
 </signal>
 <signal name="RTC_CS">
 <contactref element="U2" pad="1"/>
 <contactref element="J1" pad="1"/>
-<wire x1="4.205" y1="28.575" x2="1.27" y2="1.27" width="0" layer="19" extent="1-1"/>
+<wire x1="4.205" y1="13.335" x2="1.27" y2="1.27" width="0" layer="19" extent="1-1"/>
 </signal>
 <signal name="V_RAW">
@@
 </polygon>
 </signal>
+<signal name="BYP">
+<contactref element="U3" pad="2"/>
+<contactref element="C3" pad="1"/>
+<wire x1="-1.275" y1="-3.31" x2="3.16" y2="-8.89" width="0" layer="19" extent="1-1"/>
+</signal>
+<signal name="SCL">
+<contactref element="U3" pad="4"/>
+<contactref element="R2" pad="1"/>
+<contactref element="J3" pad="2"/>
+<wire x1="3.16" y1="-12.7" x2="2.7178" y2="-22.86" width="0" layer="19" extent="1-1"/>
+<wire x1="-1.275" y1="-4.31" x2="3.16" y2="-12.7" width="0" layer="19" extent="1-1"/>
+</signal>
+<signal name="SDA">
+<contactref element="U3" pad="6"/>
+<contactref element="R3" pad="1"/>
+<contactref element="J3" pad="1"/>
+<wire x1="-0.65" y1="-16.51" x2="-0.1778" y2="-22.86" width="0" layer="19" extent="1-1"/>
+<wire x1="-0.5" y1="-5.085" x2="-0.65" y2="-16.51" width="0" layer="19" extent="1-1"/>
+</signal>
+<signal name="SA0">
+<contactref element="U3" pad="7"/>
+<contactref element="R4" pad="1"/>
+<wire x1="0" y1="-5.085" x2="3.16" y2="-16.51" width="0" layer="19" extent="1-1"/>
+</signal>
 </signals>
