File: layer1v2/accel-sd-gyro.sch (EAGLE design)
At the start: 14 parts, among them IC2 LGD20H, U1 MMA8452Q, U2 microSD

Commit message: added headers
Parts:
- added J1, J2: (no value), SparkFun-Connectors:M12PTH
- added J3: (no value), SparkFun-Connectors:M02LOCK
Connections:
- new net INT/SQW: J1.8
- new net RTC_CS: J1.1
- new net V_RAW: J2.1
- net 3.3V: now also J2.4
- net GND: now also J1.9, J2.2
- net MISO: now also J2.10
- net MOSI: now also J2.11
- net SCK: now also J2.9
- net SCL: now also J3.2
- net SDA: now also J3.1
- net SD_CS: now also J2.12
Changed lines of the file:
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@@
 <layer number="56" name="wert" color="7" fill="1" visible="no" active="no"/>
 <layer number="57" name="tCAD" color="7" fill="1" visible="no" active="no"/>
+<layer number="59" name="tCarbon" color="7" fill="1" visible="no" active="no"/>
+<layer number="60" name="bCarbon" color="7" fill="1" visible="no" active="no"/>
 <layer number="90" name="Modules" color="5" fill="1" visible="yes" active="yes"/>
 <layer number="91" name="Nets" color="2" fill="1" visible="yes" active="yes"/>
@@
 <layer number="97" name="Info" color="7" fill="1" visible="yes" active="yes"/>
 <layer number="98" name="Guide" color="6" fill="1" visible="yes" active="yes"/>
+<layer number="99" name="SpiceOrder" color="7" fill="1" visible="yes" active="yes"/>
 <layer number="100" name="Muster" color="7" fill="1" visible="no" active="no"/>
 <layer number="101" name="Patch_Top" color="12" fill="4" visible="yes" active="yes"/>
@@
 <layer number="111" name="LPC17xx" color="7" fill="1" visible="yes" active="yes"/>
 <layer number="112" name="tSilk" color="7" fill="1" visible="yes" active="yes"/>
+<layer number="113" name="IDFDebug" color="4" fill="1" visible="yes" active="yes"/>
+<layer number="114" name="Badge_Outline" color="7" fill="1" visible="yes" active="yes"/>
+<layer number="115" name="ReferenceISLANDS" color="7" fill="1" visible="yes" active="yes"/>
 <layer number="116" name="Patch_BOT" color="9" fill="4" visible="yes" active="yes"/>
+<layer number="118" name="Rect_Pads" color="7" fill="1" visible="yes" active="yes"/>
 <layer number="121" name="_tsilk" color="7" fill="1" visible="yes" active="yes"/>
 <layer number="122" name="_bsilk" color="7" fill="1" visible="yes" active="yes"/>
@@
 <layer number="127" name="_tValues" color="7" fill="1" visible="yes" active="yes"/>
 <layer number="128" name="_bValues" color="7" fill="1" visible="yes" active="yes"/>
+<layer number="129" name="Mask" color="7" fill="1" visible="yes" active="yes"/>
 <layer number="131" name="tAdjust" color="7" fill="1" visible="no" active="yes"/>
 <layer number="132" name="bAdjust" color="7" fill="1" visible="no" active="yes"/>
@@
 <layer number="223" name="223bmp" color="24" fill="1" visible="no" active="no"/>
 <layer number="224" name="224bmp" color="25" fill="1" visible="no" active="no"/>
+<layer number="225" name="225bmp" color="7" fill="1" visible="yes" active="yes"/>
+<layer number="226" name="226bmp" color="7" fill="1" visible="yes" active="yes"/>
+<layer number="227" name="227bmp" color="7" fill="1" visible="yes" active="yes"/>
+<layer number="228" name="228bmp" color="7" fill="1" visible="yes" active="yes"/>
+<layer number="229" name="229bmp" color="7" fill="1" visible="yes" active="yes"/>
+<layer number="230" name="230bmp" color="7" fill="1" visible="yes" active="yes"/>
+<layer number="231" name="231bmp" color="7" fill="1" visible="yes" active="yes"/>
 <layer number="248" name="Housing" color="7" fill="1" visible="yes" active="yes"/>
 <layer number="249" name="Edge" color="7" fill="1" visible="yes" active="yes"/>
@@
 <layer number="251" name="SMDround" color="12" fill="11" visible="no" active="no"/>
 <layer number="254" name="cooling" color="7" fill="1" visible="yes" active="yes"/>
+<layer number="255" name="routoute" color="7" fill="1" visible="yes" active="yes"/>
 </layers>
 <schematic xreflabel="%F%N/%S.%C%R" xrefpart="/%S.%C%R">
@@
 <part name="P+8" library="SparkFun" deviceset="3.3V" device=""/>
 <part name="U2" library="SparkFun" deviceset="USD-SOCKET" device="SMD" value="microSD"/>
+<part name="J1" library="SparkFun-Connectors" deviceset="M12" device="PTH"/>
+<part name="J2" library="SparkFun-Connectors" deviceset="M12" device="PTH"/>
+<part name="J3" library="SparkFun-Connectors" deviceset="M02" device="LOCK"/>
 </parts>
 <sheets>
@@
 <attribute name="VALUE" x="168.656" y="60.706" size="1.778" layer="96"/>
 </instance>
+<instance part="J1" gate="G$1" x="7.62" y="109.22"/>
+<instance part="J2" gate="G$1" x="55.88" y="106.68" rot="R180"/>
+<instance part="J3" gate="G$1" x="30.48" y="129.54"/>
 </instances>
 <busses>
@@
 <pinref part="U2" gate="G$1" pin="VCC"/>
 <label x="200.66" y="88.9" size="1.778" layer="95"/>
+</segment>
+<segment>
+<wire x1="45.72" y1="114.3" x2="38.1" y2="114.3" width="0.1524" layer="91"/>
+<label x="38.1" y="114.3" size="1.778" layer="95"/>
+<pinref part="J2" gate="G$1" pin="4"/>
 </segment>
 </net>
@@
 <label x="200.66" y="83.82" size="1.778" layer="95"/>
 </segment>
+<segment>
+<wire x1="17.78" y1="114.3" x2="25.4" y2="114.3" width="0.1524" layer="91"/>
+<label x="20.32" y="114.3" size="1.778" layer="95"/>
+<pinref part="J1" gate="G$1" pin="9"/>
+</segment>
+<segment>
+<wire x1="45.72" y1="119.38" x2="38.1" y2="119.38" width="0.1524" layer="91"/>
+<label x="38.1" y="119.38" size="1.778" layer="95"/>
+<pinref part="J2" gate="G$1" pin="2"/>
+</segment>
 </net>
 <net name="SCL" class="0">
@@
 <pinref part="IC2" gate="G$1" pin="SCL/SPC"/>
 </segment>
+<segment>
+<pinref part="J3" gate="G$1" pin="2"/>
+<wire x1="38.1" y1="132.08" x2="43.18" y2="132.08" width="0.1524" layer="91"/>
+<label x="38.1" y="132.08" size="1.778" layer="95"/>
+</segment>
 </net>
 <net name="SDA" class="0">
@@
 <label x="144.78" y="132.08" size="1.778" layer="95"/>
 <pinref part="IC2" gate="G$1" pin="SDA/SDI/SDO"/>
+</segment>
+<segment>
+<pinref part="J3" gate="G$1" pin="1"/>
+<wire x1="38.1" y1="129.54" x2="43.18" y2="129.54" width="0.1524" layer="91"/>
+<label x="38.1" y="129.54" size="1.778" layer="95"/>
 </segment>
 </net>
@@
 <label x="198.12" y="93.98" size="1.778" layer="95"/>
 </segment>
+<segment>
+<wire x1="45.72" y1="93.98" x2="38.1" y2="93.98" width="0.1524" layer="91"/>
+<label x="38.1" y="93.98" size="1.778" layer="95"/>
+<pinref part="J2" gate="G$1" pin="12"/>
+</segment>
 </net>
 <net name="MOSI" class="0">
@@
 <label x="200.66" y="91.44" size="1.778" layer="95"/>
 </segment>
+<segment>
+<wire x1="45.72" y1="96.52" x2="38.1" y2="96.52" width="0.1524" layer="91"/>
+<label x="38.1" y="96.52" size="1.778" layer="95"/>
+<pinref part="J2" gate="G$1" pin="11"/>
+</segment>
 </net>
 <net name="SCK" class="0">
@@
 <label x="200.66" y="86.36" size="1.778" layer="95"/>
 </segment>
+<segment>
+<wire x1="45.72" y1="101.6" x2="38.1" y2="101.6" width="0.1524" layer="91"/>
+<label x="38.1" y="101.6" size="1.778" layer="95"/>
+<pinref part="J2" gate="G$1" pin="9"/>
+</segment>
 </net>
 <net name="MISO" class="0">
@@
 <label x="200.66" y="81.28" size="1.778" layer="95"/>
 </segment>
-</net>
+<segment>
+<wire x1="45.72" y1="99.06" x2="38.1" y2="99.06" width="0.1524" layer="91"/>
+<label x="38.1" y="99.06" size="1.778" layer="95"/>
+<pinref part="J2" gate="G$1" pin="10"/>
+</segment>
+</net>
+<net name="INT/SQW" class="0">
+<segment>
+<wire x1="17.78" y1="111.76" x2="25.4" y2="111.76" width="0.1524" layer="91"/>
+<label x="17.78" y="111.76" size="1.778" layer="95"/>
+<pinref part="J1" gate="G$1" pin="8"/>
+</segment>
+</net>
+<net name="RTC_CS" class="0">
+<segment>
+<wire x1="17.78" y1="93.98" x2="25.4" y2="93.98" width="0.1524" layer="91"/>
+<label x="17.78" y="93.98" size="1.778" layer="95"/>
+<pinref part="J1" gate="G$1" pin="1"/>
+</segment>
+</net>
+<net name="V_RAW" class="0">
+<segment>
+<pinref part="J2" gate="G$1" pin="1"/>
+<wire x1="45.72" y1="121.92" x2="38.1" y2="121.92" width="0.1524" layer="91"/>
+<label x="38.1" y="121.92" size="1.778" layer="95"/>
+<label x="38.1" y="121.92" size="1.778" layer="95"/>
+</segment>
+</net>
