File: uSD_test_board/uSD_test_board.sch (EAGLE design)
At the start: 6 parts

Commit message: named nets
Connections:
- net N$1 renamed CS1
- net N$10 renamed SCK2
- net N$12 renamed DO2
- net N$13 renamed CS3
- net N$14 renamed DI3
- net N$15 renamed VCC3
- net N$16 renamed SCK3
- net N$18 renamed DO3
- net N$2 renamed DI1
- net N$3 renamed VCC1
- net N$4 renamed SCK1
- net N$6 renamed DO1
- net N$7 renamed CS2
- net N$8 renamed DI2
- net N$9 renamed VCC2
- removed net N$11: J2.5, U$2.GND
- removed net N$20: J3.5, U$3.GND, U$3.SUPPORT@1, U$3.SUPPORT@2, U$3.SUPPORT@3, U$3.SUPPORT@4
- removed net N$5: J1.5, U$1.GND
- new net GND: J1.5, J2.5, J3.5, U$1.GND, U$2.GND, U$3.GND, U$3.SUPPORT@1, U$3.SUPPORT@2, U$3.SUPPORT@3, U$3.SUPPORT@4
Changed lines of the file:
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@@
 <setting verticaltext="up"/>
 </settings>
-<grid distance="0.1" unitdist="inch" unit="inch" style="lines" multiple="1" display="yes" altdistance="0.01" altunitdist="inch" altunit="inch"/>
+<grid distance="0.1" unitdist="inch" unit="inch" style="lines" multiple="1" display="no" altdistance="0.01" altunitdist="inch" altunit="inch"/>
 <layers>
 <layer number="1" name="Top" color="4" fill="1" visible="no" active="no"/>
@@
 </busses>
 <nets>
-<net name="N$1" class="0">
+<net name="CS1" class="0">
 <segment>
 <pinref part="U$1" gate="G$1" pin="CS"/>
@@
 </segment>
 </net>
-<net name="N$2" class="0">
+<net name="DI1" class="0">
 <segment>
 <pinref part="J1" gate="G$1" pin="2"/>
@@
 </segment>
 </net>
-<net name="N$3" class="0">
-<segment>
-<pinref part="J1" gate="G$1" pin="3"/>
-<pinref part="U$1" gate="G$1" pin="VCC"/>
-<wire x1="25.4" y1="86.36" x2="17.78" y2="86.36" width="0.1524" layer="91"/>
-</segment>
-</net>
-<net name="N$4" class="0">
+<net name="SCK1" class="0">
 <segment>
 <pinref part="J1" gate="G$1" pin="4"/>
@@
 </segment>
 </net>
-<net name="N$5" class="0">
+<net name="GND" class="0">
 <segment>
 <pinref part="U$1" gate="G$1" pin="GND"/>
@@
 <wire x1="17.78" y1="81.28" x2="25.4" y2="81.28" width="0.1524" layer="91"/>
 </segment>
-</net>
-<net name="N$6" class="0">
-<segment>
-<pinref part="J1" gate="G$1" pin="6"/>
-<pinref part="U$1" gate="G$1" pin="DO"/>
-<wire x1="25.4" y1="78.74" x2="17.78" y2="78.74" width="0.1524" layer="91"/>
-</segment>
-</net>
-<net name="N$7" class="0">
-<segment>
-<pinref part="J2" gate="G$1" pin="1"/>
-<pinref part="U$2" gate="G$1" pin="CS"/>
-<wire x1="73.66" y1="91.44" x2="66.04" y2="91.44" width="0.1524" layer="91"/>
-</segment>
-</net>
-<net name="N$8" class="0">
-<segment>
-<pinref part="J2" gate="G$1" pin="2"/>
-<pinref part="U$2" gate="G$1" pin="DI"/>
-<wire x1="73.66" y1="88.9" x2="66.04" y2="88.9" width="0.1524" layer="91"/>
-</segment>
-</net>
-<net name="N$9" class="0">
-<segment>
-<pinref part="U$2" gate="G$1" pin="VCC"/>
-<pinref part="J2" gate="G$1" pin="3"/>
-<wire x1="66.04" y1="86.36" x2="73.66" y2="86.36" width="0.1524" layer="91"/>
-</segment>
-</net>
-<net name="N$10" class="0">
-<segment>
-<pinref part="J2" gate="G$1" pin="4"/>
-<pinref part="U$2" gate="G$1" pin="SCK"/>
-<wire x1="73.66" y1="83.82" x2="66.04" y2="83.82" width="0.1524" layer="91"/>
-</segment>
-</net>
-<net name="N$11" class="0">
 <segment>
 <pinref part="U$2" gate="G$1" pin="GND"/>
@@
 <wire x1="66.04" y1="81.28" x2="73.66" y2="81.28" width="0.1524" layer="91"/>
 </segment>
-</net>
-<net name="N$12" class="0">
-<segment>
-<pinref part="J2" gate="G$1" pin="6"/>
-<pinref part="U$2" gate="G$1" pin="DO"/>
-<wire x1="73.66" y1="78.74" x2="66.04" y2="78.74" width="0.1524" layer="91"/>
-</segment>
-</net>
-<net name="N$13" class="0">
-<segment>
-<pinref part="J3" gate="G$1" pin="1"/>
-<pinref part="U$3" gate="G$1" pin="CS"/>
-<wire x1="127" y1="104.14" x2="119.38" y2="104.14" width="0.1524" layer="91"/>
-</segment>
-</net>
-<net name="N$14" class="0">
-<segment>
-<pinref part="J3" gate="G$1" pin="2"/>
-<pinref part="U$3" gate="G$1" pin="DI"/>
-<wire x1="127" y1="101.6" x2="119.38" y2="101.6" width="0.1524" layer="91"/>
-</segment>
-</net>
-<net name="N$15" class="0">
-<segment>
-<pinref part="J3" gate="G$1" pin="3"/>
-<pinref part="U$3" gate="G$1" pin="VCC"/>
-<wire x1="127" y1="99.06" x2="119.38" y2="99.06" width="0.1524" layer="91"/>
-</segment>
-</net>
-<net name="N$16" class="0">
-<segment>
-<pinref part="J3" gate="G$1" pin="4"/>
-<pinref part="U$3" gate="G$1" pin="SCK"/>
-<wire x1="127" y1="96.52" x2="119.38" y2="96.52" width="0.1524" layer="91"/>
-</segment>
-</net>
-<net name="N$18" class="0">
-<segment>
-<pinref part="J3" gate="G$1" pin="6"/>
-<pinref part="U$3" gate="G$1" pin="DO"/>
-<wire x1="127" y1="91.44" x2="119.38" y2="91.44" width="0.1524" layer="91"/>
-</segment>
-</net>
-<net name="N$20" class="0">
 <segment>
 <pinref part="U$3" gate="G$1" pin="SUPPORT@4"/>
@@
 </segment>
 </net>
+<net name="DO1" class="0">
+<segment>
+<pinref part="J1" gate="G$1" pin="6"/>
+<pinref part="U$1" gate="G$1" pin="DO"/>
+<wire x1="25.4" y1="78.74" x2="17.78" y2="78.74" width="0.1524" layer="91"/>
+</segment>
+</net>
+<net name="CS2" class="0">
+<segment>
+<pinref part="J2" gate="G$1" pin="1"/>
+<pinref part="U$2" gate="G$1" pin="CS"/>
+<wire x1="73.66" y1="91.44" x2="66.04" y2="91.44" width="0.1524" layer="91"/>
+</segment>
+</net>
+<net name="DI2" class="0">
+<segment>
+<pinref part="J2" gate="G$1" pin="2"/>
+<pinref part="U$2" gate="G$1" pin="DI"/>
+<wire x1="73.66" y1="88.9" x2="66.04" y2="88.9" width="0.1524" layer="91"/>
+</segment>
+</net>
+<net name="SCK2" class="0">
+<segment>
+<pinref part="J2" gate="G$1" pin="4"/>
+<pinref part="U$2" gate="G$1" pin="SCK"/>
+<wire x1="73.66" y1="83.82" x2="66.04" y2="83.82" width="0.1524" layer="91"/>
+</segment>
+</net>
+<net name="DO2" class="0">
+<segment>
+<pinref part="J2" gate="G$1" pin="6"/>
+<pinref part="U$2" gate="G$1" pin="DO"/>
+<wire x1="73.66" y1="78.74" x2="66.04" y2="78.74" width="0.1524" layer="91"/>
+</segment>
+</net>
+<net name="CS3" class="0">
+<segment>
+<pinref part="J3" gate="G$1" pin="1"/>
+<pinref part="U$3" gate="G$1" pin="CS"/>
+<wire x1="127" y1="104.14" x2="119.38" y2="104.14" width="0.1524" layer="91"/>
+</segment>
+</net>
+<net name="DI3" class="0">
+<segment>
+<pinref part="J3" gate="G$1" pin="2"/>
+<pinref part="U$3" gate="G$1" pin="DI"/>
+<wire x1="127" y1="101.6" x2="119.38" y2="101.6" width="0.1524" layer="91"/>
+</segment>
+</net>
+<net name="SCK3" class="0">
+<segment>
+<pinref part="J3" gate="G$1" pin="4"/>
+<pinref part="U$3" gate="G$1" pin="SCK"/>
+<wire x1="127" y1="96.52" x2="119.38" y2="96.52" width="0.1524" layer="91"/>
+</segment>
+</net>
+<net name="DO3" class="0">
+<segment>
+<pinref part="J3" gate="G$1" pin="6"/>
+<pinref part="U$3" gate="G$1" pin="DO"/>
+<wire x1="127" y1="91.44" x2="119.38" y2="91.44" width="0.1524" layer="91"/>
+</segment>
+</net>
+<net name="VCC1" class="0">
+<segment>
+<pinref part="U$1" gate="G$1" pin="VCC"/>
+<pinref part="J1" gate="G$1" pin="3"/>
+<wire x1="17.78" y1="86.36" x2="25.4" y2="86.36" width="0.1524" layer="91"/>
+</segment>
+</net>
+<net name="VCC2" class="0">
+<segment>
+<pinref part="U$2" gate="G$1" pin="VCC"/>
+<pinref part="J2" gate="G$1" pin="3"/>
+<wire x1="66.04" y1="86.36" x2="73.66" y2="86.36" width="0.1524" layer="91"/>
+</segment>
+</net>
+<net name="VCC3" class="0">
+<segment>
+<pinref part="U$3" gate="G$1" pin="VCC"/>
+<pinref part="J3" gate="G$1" pin="3"/>
+<wire x1="119.38" y1="99.06" x2="127" y2="99.06" width="0.1524" layer="91"/>
+</segment>
+</net>
